File: 4esc-by-martinez/4ESC v3.1.brd (EAGLE design)
At the start: 50 x 50 mm, 154 parts, among them Q1 16mhz, Q2 16mhz, Q3 16mhz, Q4 16mhz, U1 LM2842, X1 53047-06, X2 53047-03

Commit message: Schrift 4ESC verschoben
Parts:
- moved U$3 0.32 mm to (49.2, 8.73)
Changed lines of the file:
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@@
 <element name="JP1" library="SparkFun" package="1X02_NO_SILK" value="" x="9.68375" y="7.9375" rot="R180"/>
 <element name="JP2" library="SparkFun" package="1X02_NO_SILK" value="" x="40.3225" y="44.688125"/>
-<element name="U$3" library="Zeichen" package="4ESC_05MM_HOCH" value="4ESC_05MM" x="48.895" y="8.73125" rot="R90"/>
+<element name="U$3" library="Zeichen" package="4ESC_05MM_HOCH" value="4ESC_05MM" x="49.2125" y="8.73125" rot="R90"/>
 <element name="U$4" library="Zeichen" package="4ESC_05MM_HOCH" value="4ESC_05MM" x="20.32" y="3.4925" rot="MR0"/>
 </elements>
